File: hardware/universal_lights.sch (KiCad schematic (older format))
At the start: 25 parts, among them J1 entrada, J2 salida, J3 DIP-BLACK-MALE-HEADER_2X3P-2.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, J4 Conn_01x08, J5 Conn_01x02, Q1 NPN, U1 ATTINY88-AU

Commit message: WIP del atmega 328 para ADCtouch
Parts:
- removed U1: ATTINY88-AU, Housings_QFP:TQFP-32_7x7mm_Pitch0.8mm, symbol ATTINY88-AU
- added U?: ATmega328P-AU, Package_QFP:TQFP-32_7x7mm_P0.8mm, symbol MCU_Microchip_ATmega:ATmega328P-AU
- added Y?: 16Mhz, symbol SeeedOPL-Crystal_Oscillator-2016:SMD-RESONATOR-16MHZ-15PF-0.5%-40R_3P-3.2X1.3MM_
- C1: symbol CERAMIC-2.2UF-10V-10%-X7R_0603_ -> universal_lights-rescue:CERAMIC-2.2UF-10V-10%-X7R_0603_
- D1, D2, D3, D4, D5: symbol SMD-LED-CLEAR-BLUE_0603_ -> universal_lights-rescue:SMD-LED-CLEAR-BLUE_0603_
- J1, J2: symbol DIP-BLACK-MALE-HEADER-R_A_3P-2.54-90D_ -> universal_lights-rescue:DIP-BLACK-MALE-HEADER-R_A_3P-2.54-90D_
- J3: symbol DIP-BLACK-MALE-HEADER_2X3P-2.54) -> universal_lights-rescue:DIP-BLACK-MALE-HEADER_2X3P-2.54)
- J4: symbol Conn_01x08 -> universal_lights-rescue:Conn_01x08
- J5: symbol Conn_01x02 -> universal_lights-rescue:Conn_01x02
- LED1, LED2, LED3, LED4, LED5: symbol WS2812B -> universal_lights-rescue:WS2812B
- Q1: symbol SMD-TRANSISTORS-NPN-25V-500MA-S9013_SOT-23_ -> universal_lights-rescue:SMD-TRANSISTORS-NPN-25V-500MA-S9013_SOT-23_
- R1, R2, R3, R4, R5, R6: symbol SMD-RES-220R-5%-1_10W_0603_ -> universal_lights-rescue:SMD-RES-220R-5%-1_10W_0603_
- R9: symbol SMD-RES-1K-1%-1_10W_0603_ -> universal_lights-rescue:SMD-RES-1K-1%-1_10W_0603_
Connections:
- wire segments 67 -> 81
- no-connect marks 14 -> 0
Other:
- moved on the sheet: R5

Commit message: instalado atmega 328, ajustados agujeros de montaje, cambio silk versión
Parts:
- Y1: renamed from Y?; footprint (none) -> SeeedOPL-Crystal Oscillator-2016:X3-SMD-3.6X1.3X0.8MM
- gave numbers to parts that had none: 1
Connections:
- no-connect marks 0 -> 9
Changed lines of the file:
@@
 	3500 4550 3750 4550
 $Comp
-L MCU_Microchip_ATmega:ATmega328P-AU U?
+L MCU_Microchip_ATmega:ATmega328P-AU U1
 U 1 1 5B0D318C
 P 2300 4250
-F 0 "U?" H 2700 2800 50  0000 C CNN
+F 0 "U1" H 2700 2800 50  0000 C CNN
 F 1 "ATmega328P-AU" H 2900 2700 50  0000 C CNN
 F 2 "Package_QFP:TQFP-32_7x7mm_P0.8mm" H 2300 4250 50  0001 C CIN
@@
 	2900 3550 3500 3550
 $Comp
-L SeeedOPL-Crystal_Oscillator-2016:SMD-RESONATOR-16MHZ-15PF-0.5%-40R_3P-3.2X1.3MM_ Y?
+L SeeedOPL-Crystal_Oscillator-2016:SMD-RESONATOR-16MHZ-15PF-0.5%-40R_3P-3.2X1.3MM_ Y1
 U 1 1 5B0EBA8F
 P 3350 3750
-F 0 "Y?" V 3450 3400 45  0000 L CNN
+F 0 "Y1" V 3450 3400 45  0000 L CNN
 F 1 "16Mhz" V 3250 3300 45  0000 L CNN
-F 2 "" H 3350 3750 50  0001 C CNN
+F 2 "SeeedOPL-Crystal Oscillator-2016:X3-SMD-3.6X1.3X0.8MM" H 3350 3750 50  0001 C CNN
 F 3 "" H 3350 3750 50  0001 C CNN
 F 4 "CSTCE16M0V53-R0" H 3380 3900 20  0001 C CNN "MPN"
@@
 	3050 3850 3350 3850
 $Comp
-L universal_lights-rescue:GND #PWR?
+L universal_lights-rescue:GND #PWR0101
 U 1 1 5B0F15A0
 P 3650 3750
-F 0 "#PWR?" H 3650 3500 50  0001 C CNN
+F 0 "#PWR0101" H 3650 3500 50  0001 C CNN
 F 1 "GND" H 3650 3600 50  0000 C CNN
 F 2 "" H 3650 3750 50  0001 C CNN
@@
 Wire Wire Line
 	1700 3050 1700 2950
+NoConn ~ 1700 3250
+NoConn ~ 1700 3350
+NoConn ~ 2900 4250
+NoConn ~ 2900 4750
+NoConn ~ 2900 4850
+NoConn ~ 2900 5150
+NoConn ~ 2900 5250
+NoConn ~ 2900 5350
+NoConn ~ 2900 5450
 $EndSCHEMATC

Commit message: añado 470R a entrada datos led, muevo cristal para que sea mas facil de soldar
Parts:
- added R7: 470, SeeedOPL-Resistor-2016:R0603, symbol universal_lights-rescue:SMD-RES-220R-5%-1_10W_0603_
Connections:
- wire segments 81 -> 82
Changed lines of the file:
@@
 	1    0    0    -1
 $EndComp
-Text Label 3500 3050 2    60   ~ 0
+Text Label 3800 3050 2    60   ~ 0
 datos_led_in
 Text Label 3500 3150 2    60   ~ 0
@@
 Connection ~ 2300 2700
 Wire Wire Line
-	2900 3050 3500 3050
-Wire Wire Line
 	2900 3250 3500 3250
 Wire Wire Line
@@
 NoConn ~ 2900 5350
 NoConn ~ 2900 5450
+$Comp
+L universal_lights-rescue:SMD-RES-220R-5%-1_10W_0603_ R7
+U 1 1 5B0D9833
+P 3100 3050
+F 0 "R7" H 2950 3100 45  0000 L BNN
+F 1 "470" H 2950 2950 45  0000 L BNN
+F 2 "SeeedOPL-Resistor-2016:R0603" H 3100 3050 40  0001 C CNN
+F 3 "" H 3100 3050 40  0001 C CNN
+F 4 "RC0603JR-07220RL" H 3130 3200 20  0001 C CNN "MPN"
+F 5 "301010163" H 3130 3200 20  0001 C CNN "SKU"
+	1    3100 3050
+	1    0    0    -1
+$EndComp
+Wire Wire Line
+	2900 3050 2950 3050
+Wire Wire Line
+	3800 3050 3250 3050
 $EndSCHEMATC
